Commit message: dodana roka in stvari iz dis_tutorial7

File: urdf/standard/turtlebot4.urdf.xacro (robot description, xacro)
@@ -2,11 +2,13 @@
 <robot name="turtlebot4" xmlns:xacro="http://ros.org/wiki/xacro">
   <!-- Base create3 model -->
-  <xacro:include filename="$(find irobot_create_description)/urdf/create3.urdf.xacro" />
-  <xacro:include filename="$(find dis_tutorial3)/urdf/sensors/rplidar.urdf.xacro" />
-  <xacro:include filename="$(find dis_tutorial3)/urdf/sensors/oakd.urdf.xacro" />
-  <xacro:include filename="$(find dis_tutorial3)/urdf/sensors/camera_bracket.urdf.xacro" />
-  <xacro:include filename="$(find dis_tutorial3)/urdf/standard/tower_standoff.urdf.xacro" />
-  <xacro:include filename="$(find dis_tutorial3)/urdf/standard/tower_sensor_plate.urdf.xacro" />
-  <xacro:include filename="$(find dis_tutorial3)/urdf/standard/weight_block.urdf.xacro" />
+  <xacro:include filename="$(find rins_robot)/urdf/create/create3.urdf.xacro" />
+  <xacro:include filename="$(find rins_robot)/urdf/sensors/rplidar.urdf.xacro" />
+  <xacro:include filename="$(find rins_robot)/urdf/sensors/oakd.urdf.xacro" />
+  <xacro:include filename="$(find rins_robot)/urdf/sensors/top_camera.urdf.xacro" />
+  <xacro:include filename="$(find rins_robot)/urdf/sensors/camera_bracket.urdf.xacro" />
+  <xacro:include filename="$(find rins_robot)/urdf/standard/tower_standoff.urdf.xacro" />
+  <xacro:include filename="$(find rins_robot)/urdf/standard/tower_sensor_plate.urdf.xacro" />
+  <xacro:include filename="$(find rins_robot)/urdf/standard/weight_block.urdf.xacro" />
+  <xacro:include filename="$(find rins_robot)/urdf/arm/arm.urdf.xacro" />
   <!-- Mechanical properties -->
   <xacro:property name="shell_z_offset"                value="${3*cm2m}" />
@@ -101,4 +103,22 @@
     <origin xyz="${oakd_pro_x_offset} ${oakd_pro_y_offset} ${oakd_pro_z_offset}"/>
   </xacro:oakd>
+  <xacro:simple_arm parent_link="tower_sensor_plate">
+    <origin xyz="0 0 0.01" rpy="0 0 0"/>
+  </xacro:simple_arm>
+  <xacro:top_camera name="top_camera" model="pro" parent_link="arm_wrist_link">
+    <origin xyz="0 0 0.065" rpy="0 -${pi/2} 0"/>
+  </xacro:top_camera>
+  <gazebo>
+    <plugin filename="libgz_ros2_control-system.so" name="gz_ros2_control::GazeboSimROS2ControlPlugin">
+      <parameters>$(find rins_robot)/config/all_controls_jtc.yaml</parameters>
+      <ros>
+        <remapping>~/odom:=odom</remapping>
+        <remapping>/tf:=tf</remapping>
+        <remapping>/tf_static:=tf_static</remapping>
+        <remapping>/diagnostics:=diagnostics</remapping>
+        <namespace>$(arg namespace)</namespace>
+      </ros>
+    </plugin>
+  </gazebo>
   <!-- Base footprint for navigation -->
   <link name="base_footprint" />
